Commit message: gazebo

File: urdf/theclaw.urdf (robot description, URDF)
Before this commit: robot omniplatform, 4 links, 3 joints
Links:
- link base_link: geometry collision cylinder length=0.6 radius=0.2; visual mesh filename=package://theclaw/urdf/model/Platform.stl scale=${model_scale}
- link wheel1: geometry visual mesh filename=package://theclaw/urdf/model/Omniwheel.stl scale=${model_scale}
- link wheel2: geometry visual mesh filename=package://theclaw/urdf/model/Omniwheel.stl scale=${model_scale}
- link wheel3: geometry visual mesh filename=package://theclaw/urdf/model/Omniwheel.stl scale=${model_scale}
