Commit message: lidar

File: urdf/common_properties.xacro (robot description, xacro)
@@ -1,4 +1,13 @@
 <?xml version="1.0" ?>
 <robot name="xacro_properties" xmlns:xacro="http://ros.org/wiki/xacro">
+    <xacro:macro name="inertial_cylinder" params="mass radius length *origin">
+        <inertial>
+            <xacro:insert_block name="origin" />
+            <mass value="${mass}" />
+            <inertia ixx="${1/12*mass*(3*radius*radius+length*length)}" ixy="0.0" ixz="0.0"
+                     iyy="${1/12*mass*(3*radius*radius+length*length)}" iyz="0.0"
+                     izz="${0.5*mass*radius*radius}" />
+        </inertial>
+    </xacro:macro>
   <material name="black">
       <color rgba="0.0 0.0 0.0 1.0"/>

File: urdf/theclaw.gazebo.xacro (robot description, xacro)
@@ -3,7 +3,4 @@
   <gazebo reference="base_link">
     <material>Gazebo/White</material>
-  </gazebo>
-  <gazebo reference="camera_link">
-    <material>Gazebo/Green</material>
   </gazebo>
   <gazebo reference="wheel1">
@@ -17,4 +14,5 @@
   </gazebo>
   <gazebo reference="camera_link">
+    <material>Gazebo/Green</material>
     <sensor type="camera" name="camera1">
       <update_rate>30.0</update_rate>
@@ -42,5 +40,5 @@
         <alwaysOn>true</alwaysOn>
         <updateRate>0.0</updateRate>
-        <cameraName>jetbot/camera</cameraName>
+        <cameraName>camera</cameraName>
         <imageTopicName>image_raw</imageTopicName>
         <cameraInfoTopicName>camera_info</cameraInfoTopicName>
@@ -55,3 +53,33 @@
     </sensor>
   </gazebo>
+  <gazebo reference="laser_head">
+    <material>Gazebo/Red</material>
+    <sensor type="ray" name="laser_sensor">
+      <pose>0 0 0 0 0 0</pose>
+      <visualize>false</visualize>
+      <update_rate>10</update_rate>
+      <ray>
+        <scan>
+          <horizontal>
+            <samples>1470</samples>
+            <min_angle>-3.14</min_angle>
+            <max_angle>3.14</max_angle>
+          </horizontal>
+        </scan>
+        <range>
+          <min>0.2</min>
+          <max>10.0</max>
+        </range>
+        <noise>
+          <type>gaussian</type>
+          <mean>0.0</mean>
+          <stddev>0.01</stddev>
+        </noise>
+      </ray>
+      <plugin name="gazebo_ros_laser_controller" filename="libgazebo_ros_laser.so">
+        <topicName>scan</topicName>
+        <frameName>laser_head</frameName>
+      </plugin>
+    </sensor>
+  </gazebo>
 </robot>

File: urdf/theclaw.urdf.xacro (robot description, xacro)
@@ -10,4 +10,5 @@
         <origin xyz="0.0 0.0 0.0" rpy=" 0 0 0"/>
     </joint>
+    <!-- Base -->
     <link name="base_link">
         <visual>
@@ -31,4 +32,5 @@
         </inertial>
     </link>
+    <!-- Camera -->
     <link name="camera_link">
         <inertial>
@@ -38,5 +40,5 @@
         </inertial>
         <visual>
-            <origin rpy="0  0  0" xyz="0  0  0" />
+            <origin rpy="0 0 0" xyz="0 0 0" />
             <geometry>
                 <box size="0.005 0.05 0.05" />
@@ -47,5 +49,38 @@
         <parent link="base_link" />
         <child link="camera_link" />
-        <origin rpy="0 0.25 0" xyz="0.055 0 0.0857" />
+        <origin rpy="0 0.2 0" xyz="0.055 0 0.07" />
+    </joint>
+    <!-- Laser -->
+    <link name="laser_base">
+        <visual>
+            <origin rpy="0 0 0" xyz="0 0 ${0.0186/2}" />
+            <geometry>
+                <cylinder radius="${0.076/2}" length="0.0186" />
+            </geometry>
+        </visual>
+        <xacro:inertial_cylinder mass="0.1" radius="${0.076/2}" length="0.0186">
+            <origin rpy="0 0 0" xyz="0 0 ${0.0186/2}" />
+        </xacro:inertial_cylinder>
+    </link>
+    <link name="laser_head">
+        <visual>
+            <origin rpy="0 0 0" xyz="0 0 ${(0.041-0.0196)/2}" />
+            <geometry>
+                <cylinder radius="${0.0725/2}" length="${0.041-0.0196}"/>
+            </geometry>
+        </visual>
+        <xacro:inertial_cylinder mass="0.1" radius="${0.0725/2}" length="${0.041-0.0196}">
+            <origin rpy="0 0 0" xyz="0 0 ${0.0186/2}" />
+        </xacro:inertial_cylinder>
+    </link>
+    <joint name="laser_base_joint" type="fixed">
+        <parent link="base_link" />
+        <child link="laser_base" />
+        <origin rpy="0 0 0" xyz="0 0 0.10" />
+    </joint>
+    <joint name="laser_head_joint" type="fixed">
+        <parent link="laser_base" />
+        <child link="laser_head" />
+        <origin rpy="0 0 0" xyz="0 0 0.0196" />
     </joint>
     <!-- Wheels !-->

Commit message: new robot

File: urdf/common_properties.xacro (robot description, xacro)
@@ -1,13 +1,88 @@
 <?xml version="1.0" ?>
 <robot name="xacro_properties" xmlns:xacro="http://ros.org/wiki/xacro">
-    <xacro:macro name="inertial_cylinder" params="mass radius length *origin">
-        <inertial>
-            <xacro:insert_block name="origin" />
-            <mass value="${mass}" />
-            <inertia ixx="${1/12*mass*(3*radius*radius+length*length)}" ixy="0.0" ixz="0.0"
-                     iyy="${1/12*mass*(3*radius*radius+length*length)}" iyz="0.0"
-                     izz="${0.5*mass*radius*radius}" />
-        </inertial>
-    </xacro:macro>
+  <xacro:macro name="inertial_cylinder" params="mass radius length *origin">
+    <inertial>
+      <xacro:insert_block name="origin" />
+      <mass value="${mass}" />
+      <inertia ixx="${1/12*mass*(3*radius*radius+length*length)}" ixy="0.0" ixz="0.0"
+               iyy="${1/12*mass*(3*radius*radius+length*length)}" iyz="0.0"
+               izz="${0.5*mass*radius*radius}" />
+    </inertial>
+  </xacro:macro>
+  <xacro:macro name="inertial_box" params="mass sx sy sz *origin">
+    <inertial>
+      <xacro:insert_block name="origin" />
+      <mass value="${mass}" />
+      <inertia ixx="${1/12*mass*(sy*sy+sz*sz)}" ixy="0.0" ixz="0.0"
+               iyy="${1/12*mass*(sx*sx+sz*sz)}" iyz="0.0"
+               izz="${1/12*mass*(sx*sx+sy*sy)}" />
+    </inertial>
+  </xacro:macro>
+  <xacro:macro name="inertial_sphere" params="mass radius *origin">
+    <inertial>
+      <xacro:insert_block name="origin" />
+      <mass value="${mass}" />
+      <inertia ixx="${2/5*mass*radius*radius}" ixy="0.0" ixz="0.0"
+               iyy="${2/5*mass*radius*radius}" iyz="0.0"
+               izz="${2/5*mass*radius*radius}" />
+    </inertial>
+  </xacro:macro>
+  <xacro:macro name="box_link" params="name mass sx sy sz">
+    <link name="${name}">
+      <visual>
+        <origin rpy="0 0 0"/>
+        <geometry>
+          <box size="${sx} ${sy} ${sz}" />
+        </geometry>
+      </visual>
+      <collision>
+        <origin rpy="0 0 0"/>
+        <geometry>
+          <box size="${sx} ${sy} ${sz}" />
+        </geometry>
+      </collision>
+      <xacro:inertial_box mass="${mass}" sx="${sx}" sy="${sy}" sz="${sz}">
+        <origin rpy="0 0 0"/>
+      </xacro:inertial_box>
+    </link>
+  </xacro:macro>
+  <xacro:macro name="cylinder_link" params="name mass radius length">
+    <link name="${name}">
+      <visual>
+        <origin rpy="0 0 0"/>
+        <geometry>
+          <cylinder radius="${radius}" length="${length}" />
+        </geometry>
+      </visual>
+      <collision>
+        <origin rpy="0 0 0"/>
+        <geometry>
+          <cylinder radius="${radius}" length="${length}" />
+        </geometry>
+      </collision>
+      <xacro:inertial_cylinder mass="${mass}" radius="${radius}" length="${length}">
+        <origin rpy="0 0 0"/>
+      </xacro:inertial_cylinder>
+    </link>
+  </xacro:macro>
+  <xacro:macro name="sphere_link" params="name mass radius">
+    <link name="${name}">
+      <visual>
+        <origin rpy="0 0 0"/>
+        <geometry>
+          <sphere radius="${radius}" />
+        </geometry>
+      </visual>
+      <collision>
+        <origin rpy="0 0 0"/>
+        <geometry>
+          <sphere radius="${radius}" />
+        </geometry>
+      </collision>
+      <xacro:inertial_sphere mass="${mass}" radius="${radius}">
+        <origin rpy="0 0 0"/>
+      </xacro:inertial_sphere>
+    </link>
+  </xacro:macro>
   <material name="black">
       <color rgba="0.0 0.0 0.0 1.0"/>

File: urdf/theclaw.gazebo.xacro (robot description, xacro)
@@ -22,12 +22,9 @@
     </sensor>
   </gazebo>
-  <gazebo reference="wheel1">
-    <material>Gazebo/White</material>
+  <gazebo reference="wheel_left_link">
+    <material>Gazebo/Grass</material>
   </gazebo>
-  <gazebo reference="wheel2">
-    <material>Gazebo/White</material>
-  </gazebo>
-  <gazebo reference="wheel3">
-    <material>Gazebo/White</material>
+  <gazebo reference="wheel_right_link">
+    <material>Gazebo/Grass</material>
   </gazebo>
   <gazebo reference="camera_link">
@@ -38,11 +35,11 @@
         <horizontal_fov>1.3962634</horizontal_fov>
         <image>
-          <width>800</width>
-          <height>800</height>
+          <width>640</width>
+          <height>640</height>
           <format>R8G8B8</format>
         </image>
         <clip>
           <near>0.02</near>
-          <far>300</far>
+          <far>100</far>
         </clip>
         <noise>
@@ -71,5 +68,5 @@
     </sensor>
   </gazebo>
-  <gazebo reference="laser_head">
+  <gazebo reference="laser_link">
     <material>Gazebo/Red</material>
     <sensor type="ray" name="laser_sensor">
@@ -86,5 +83,5 @@
         </scan>
         <range>
-          <min>0.05</min>
+          <min>0.20</min>
           <max>10.0</max>
         </range>

File: urdf/theclaw.urdf.xacro (robot description, xacro)
@@ -4,42 +4,14 @@
     <xacro:include filename="$(find theclaw)/urdf/theclaw.gazebo.xacro"/>
     <xacro:property name="model_scale" value="0.01 0.01 0.01" />
-    <link name="base_footprint"/>
-    <joint name="base_joint" type="fixed">
-        <parent link="base_footprint"/>
+    <link name="origin"/>
+    <joint name="origin_joint" type="fixed">
+        <parent link="origin"/>
         <child link="base_link"/>
-        <origin xyz="0.0 0.0 0.025" rpy="0 0 0"/>
+        <origin xyz="0.0 0.0 0.0" rpy="0 0 0"/>
     </joint>
     <!-- Base -->
-    <link name="base_link">
-        <visual>
-            <origin rpy="0 0 ${pi/2}"/>
-            <geometry>
-                <mesh filename="package://theclaw/urdf/meshes/Platform.stl" scale="${model_scale}"/>
-            </geometry>
-        </visual>
-        <collision>
-            <origin rpy="0 0 ${pi/2}"/>
-            <geometry>
-                <cylinder radius="0.060" length="0.02" />
-            </geometry>
-        </collision>
-        <xacro:inertial_cylinder mass="0.200" radius="0.060" length="0.02">
-            <origin rpy="0 0 ${pi/2}"/>
-        </xacro:inertial_cylinder>
-    </link>
+    <xacro:box_link name="base_link" mass="0.050" sx="0.150" sy="0.100" sz="0.005" />
     <!-- Camera -->
-    <link name="camera_link">
-        <inertial>
-            <mass value="0.01" />
-            <origin rpy="0 0 0" xyz="0 0 0" />
-            <inertia ixx="0" ixy="0" ixz="0" iyy="0" iyz="0" izz="0" />
-        </inertial>
-        <visual>
-            <origin rpy="0 0 0" xyz="0 0 0" />
-            <geometry>
-                <box size="0.005 0.05 0.05" />
-            </geometry>
-        </visual>
-    </link>
+    <xacro:box_link name="camera_link" mass="0.001" sx="0.005" sy="0.050" sz="0.050" />
     <joint name="camera_joint" type="fixed">
         <parent link="base_link" />
@@ -48,60 +20,23 @@
     </joint>
     <!-- Laser -->
-    <link name="laser_base">
-        <visual>
-            <origin rpy="0 0 0" xyz="0 0 ${0.0186/2}" />
-            <geometry>
-                <cylinder radius="${0.076/2}" length="0.0186" />
-            </geometry>
-        </visual>
-        <xacro:inertial_cylinder mass="0.050" radius="${0.076/2}" length="0.0186">
-            <origin rpy="0 0 0" xyz="0 0 ${0.0186/2}" />
-        </xacro:inertial_cylinder>
-    </link>
-    <link name="laser_head">
-        <visual>
-            <origin rpy="0 0 0" xyz="0 0 ${(0.041-0.0196)/2}" />
-            <geometry>
-                <cylinder radius="${0.0725/2}" length="${0.041-0.0196}"/>
-            </geometry>
-        </visual>
-        <xacro:inertial_cylinder mass="0.050" radius="${0.0725/2}" length="${0.041-0.0196}">
-            <origin rpy="0 0 0" xyz="0 0 ${0.0186/2}" />
-        </xacro:inertial_cylinder>
-    </link>
+    <xacro:cylinder_link name="laser_base_link" mass="0.050" radius="${0.076/2}" length="0.0186" />
+    <xacro:cylinder_link name="laser_link" mass="0.050" radius="${0.0725/2}" length="${0.041-0.0196}" />
     <joint name="laser_base_joint" type="fixed">
         <parent link="base_link" />
-        <child link="laser_base" />
-        <origin rpy="0 0 0" xyz="0 0 0.10" />
+        <child link="laser_base_link" />
+        <origin rpy="0 0 0" xyz="0 0 0.050" />
     </joint>
     <joint name="laser_head_joint" type="fixed">
-        <parent link="laser_base" />
-        <child link="laser_head" />
-        <origin rpy="0 0 0" xyz="0 0 0.0196" />
+        <parent link="laser_base_link" />
+        <child link="laser_link" />
+        <origin rpy="0 0 0" xyz="0 0 ${0.0186/2+(0.041-0.0196)/2}" />
     </joint>
     <!-- Wheels !-->
     <xacro:macro name="wheel" params="name *origin">
-        <link name="${name}_link">
-            <visual>
-                <origin rpy="0 ${pi/2} 0"/>
-                <geometry>
-                    <mesh filename="package://theclaw/urdf/meshes/Omniwheel.stl" scale="${model_scale}"/>
-                </geometry>
-            </visual>
-            <collision>
-                <origin rpy="0 ${pi/2} 0"/>
-                <geometry>
-                    <cylinder radius="0.025" length="0.025" />
-                </geometry>
-            </collision>
-            <xacro:inertial_cylinder mass="0.020" radius="0.025" length="0.025">
-                <origin rpy="0 ${pi/2} 0"/>
-            </xacro:inertial_cylinder>
-        </link>
+        <xacro:cylinder_link name="${name}_link" mass="0.035" radius="0.040" length="0.017" />
         <joint name="${name}_joint" type="continuous">
             <xacro:insert_block name="origin" />
-            <parent link="base_link"/>
-            <child link="${name}_link"/>
-            <limit velocity="10.0" effort="1.0"/>
+            <parent link="base_link" />
+            <child link="${name}_link" />
         </joint>
         <transmission name="${name}_tran">
@@ -110,5 +45,5 @@
                 <hardwareInterface>hardware_interface/VelocityJointInterface</hardwareInterface>
             </joint>
-            <actuator name="${name}_motor">
+            <actuator name="${name}_act">
                 <hardwareInterface>hardware_interface/VelocityJointInterface</hardwareInterface>
                 <mechanicalReduction>1</mechanicalReduction>
@@ -116,12 +51,37 @@
         </transmission>
     </xacro:macro>
-    <xacro:wheel name="wheel1">
-        <origin xyz="0.077647 0 0" rpy="0 0 0"/>
+    <xacro:wheel name="wheel_left">
+        <origin xyz="0 ${-0.050-0.017/2} 0" rpy="${pi/2} 0 0" />
     </xacro:wheel>
-    <xacro:wheel name="wheel2">
-        <origin xyz="${cos(2*pi/3)*0.077647 - sin(2*pi/3)*0} ${sin(2*pi/3)*0.077647 + cos(2*pi/3)*0} 0" rpy="0 0 ${2*pi/3}"/>
+    <xacro:wheel name="wheel_right">
+        <origin xyz="0 ${0.050+0.017/2} 0" rpy="${-pi/2} 0 0" />
     </xacro:wheel>
-    <xacro:wheel name="wheel3">
-        <origin xyz="${cos(2*pi/3*2)*0.077647 - sin(2*pi/3*2)*0} ${sin(2*pi/3*2)*0.077647 + cos(2*pi/3*2)*0} 0" rpy="0 0 ${2*pi/3*2}"/>
-    </xacro:wheel>
+    <!-- Skids -->
+    <xacro:macro name="skid" params="name *origin">
+        <xacro:sphere_link name="${name}_link1" mass="0.001" radius="0.001" />
+        <joint name="${name}_joint1" type="continuous">
+            <xacro:insert_block name="origin" />
+            <parent link="base_link" />
+            <child link="${name}_link1" />
+            <axis xyz="1 0 0" />
+        </joint>
+        <xacro:sphere_link name="${name}_link2" mass="0.001" radius="0.001" />
+        <joint name="${name}_joint2" type="continuous">
+            <parent link="${name}_link1" />
+            <child link="${name}_link2" />
+            <axis xyz="0 1 0" />
+        </joint>
+        <xacro:sphere_link name="${name}_link3" mass="0.010" radius="0.010" />
+        <joint name="${name}_joint3" type="continuous">
+            <parent link="${name}_link2" />
+            <child link="${name}_link3" />
+            <axis xyz="0 0 1" />
+        </joint>
+    </xacro:macro>
+    <xacro:skid name="skid_front">
+        <origin xyz="0.050 0 ${-0.040+0.010+0.001}" />
+    </xacro:skid>
+    <xacro:skid name="skid_rear">
+        <origin xyz="-0.050 0 ${-0.040+0.010+0.001}" />
+    </xacro:skid>
 </robot>
