Commit message: motors

File: urdf/theclaw.gazebo.xacro (robot description, xacro)
@@ -83,3 +83,8 @@
     </sensor>
   </gazebo>
+  <gazebo>
+    <plugin name="gazebo_ros_control" filename="libgazebo_ros_control.so">
+      <robotNamespace>/theclaw</robotNamespace>
+    </plugin>
+  </gazebo>
 </robot>

File: urdf/theclaw.urdf.xacro (robot description, xacro)
@@ -103,5 +103,16 @@
             <parent link="base_link"/>
             <child link="${name}_link"/>
+            <limit velocity="2" effort="0.01"/>
         </joint>
+        <transmission name="${name}_tran">
+            <type>transmission_interface/SimpleTransmission</type>
+            <joint name="${name}_joint">
+                <hardwareInterface>hardware_interface/EffortJointInterface</hardwareInterface>
+            </joint>
+            <actuator name="${name}_motor">
+                <hardwareInterface>hardware_interface/EffortJointInterface</hardwareInterface>
+                <mechanicalReduction>1</mechanicalReduction>
+            </actuator>
+        </transmission>
     </xacro:macro>
     <xacro:wheel name="wheel1">

Commit message: better diff drive

File: urdf/theclaw.gazebo.xacro (robot description, xacro)
@@ -23,8 +23,8 @@
   </gazebo>
   <gazebo reference="wheel_left_link">
-    <material>Gazebo/Grass</material>
+    <material>Gazebo/Green</material>
   </gazebo>
   <gazebo reference="wheel_right_link">
-    <material>Gazebo/Grass</material>
+    <material>Gazebo/Red</material>
   </gazebo>
   <gazebo reference="camera_link">
@@ -100,5 +100,4 @@
   <gazebo>
     <plugin name="gazebo_ros_control" filename="libgazebo_ros_control.so">
-      <robotNamespace>/theclaw</robotNamespace>
     </plugin>
   </gazebo>

File: urdf/theclaw.urdf.xacro (robot description, xacro)
@@ -40,4 +40,5 @@
             <child link="${name}_link" />
             <axis xyz="0 0 1" />
+            <limit effort="0.07" velocity="16" />
         </joint>
         <transmission name="${name}_tran">
@@ -53,8 +54,8 @@
     </xacro:macro>
     <xacro:wheel name="wheel_left">
-        <origin xyz="0 ${-0.050-0.017/2} 0" rpy="${-pi/2} 0 0" />
+        <origin xyz="0 ${0.050+0.017/2} 0" rpy="${-pi/2} 0 0" />
     </xacro:wheel>
     <xacro:wheel name="wheel_right">
-        <origin xyz="0 ${0.050+0.017/2} 0" rpy="${pi/2} 0 ${pi}" />
+        <origin xyz="0 ${-0.050-0.017/2} 0" rpy="${pi/2} 0 ${pi}" />
     </xacro:wheel>
     <!-- Skids -->
