Commit message: better model

File: urdf/theclaw.urdf.xacro (robot description, xacro)
@@ -8,5 +8,5 @@
         <parent link="base_footprint"/>
         <child link="base_link"/>
-        <origin xyz="0.0 0.0 0.0" rpy=" 0 0 0"/>
+        <origin xyz="0.0 0.0 0.025" rpy=" 0 0 0"/>
     </joint>
     <!-- Base -->
@@ -21,19 +21,15 @@
             <origin rpy="0 0 ${pi/2}"/>
             <geometry>
-                <mesh filename="package://theclaw/urdf/meshes/Platform.stl" scale="${model_scale}"/>
+                <cylinder radius="0.060" length="0.02" />
             </geometry>
         </collision>
-        <inertial>
+        <xacro:inertial_cylinder mass="0.200" radius="0.060" length="0.02">
             <origin rpy="0 0 ${pi/2}"/>
-            <mass value="0.100"/>
-            <inertia ixx="1.17545509e-04" ixy="-2.22398736e-12" ixz="6.88895872e-13"
-                     iyy="1.00073449e-04" iyz="-4.90557377e-07"
-                     izz="2.10087193e-04" />
-        </inertial>
+        </xacro:inertial_cylinder>
     </link>
     <!-- Camera -->
     <link name="camera_link">
         <inertial>
-            <mass value="0.1" />
+            <mass value="0.01" />
             <origin rpy="0 0 0" xyz="0 0 0" />
             <inertia ixx="0" ixy="0" ixz="0" iyy="0" iyz="0" izz="0" />
@@ -59,5 +55,5 @@
             </geometry>
         </visual>
-        <xacro:inertial_cylinder mass="0.1" radius="${0.076/2}" length="0.0186">
+        <xacro:inertial_cylinder mass="0.050" radius="${0.076/2}" length="0.0186">
             <origin rpy="0 0 0" xyz="0 0 ${0.0186/2}" />
         </xacro:inertial_cylinder>
@@ -70,5 +66,5 @@
             </geometry>
         </visual>
-        <xacro:inertial_cylinder mass="0.1" radius="${0.0725/2}" length="${0.041-0.0196}">
+        <xacro:inertial_cylinder mass="0.050" radius="${0.0725/2}" length="${0.041-0.0196}">
             <origin rpy="0 0 0" xyz="0 0 ${0.0186/2}" />
         </xacro:inertial_cylinder>
@@ -85,81 +81,36 @@
     </joint>
     <!-- Wheels !-->
-    <link name="wheel1">
-        <visual>
-            <origin rpy="0 ${pi/2} 0"/>
-            <geometry>
-                <mesh filename="package://theclaw/urdf/meshes/Omniwheel.stl" scale="${model_scale}"/>
-            </geometry>
-        </visual>
-        <collision>
-        <origin rpy="0 ${pi/2} 0"/>
-            <geometry>
-                <mesh filename="package://theclaw/urdf/meshes/Omniwheel.stl" scale="${model_scale}"/>
-            </geometry>
-        </collision>
-        <inertial>
-            <origin rpy="0 ${pi/2} 0"/>
-            <mass value="0.020"/>
-            <inertia ixx="4.05491236e-06" ixy="-2.30614871e-09" ixz="-3.59024381e-09"
-                     iyy="4.05452187e-06" iyz="2.37778687e-09"
-                     izz="5.84593279e-06" />
-        </inertial>
-    </link>
-    <link name="wheel2">
-        <visual>
-            <origin rpy="0 ${pi/2} 0"/>
-            <geometry>
-                <mesh filename="package://theclaw/urdf/meshes/Omniwheel.stl" scale="${model_scale}"/>
-            </geometry>
-        </visual>
-        <collision>
-           <origin rpy="0 ${pi/2} 0"/>
-            <geometry>
-                <mesh filename="package://theclaw/urdf/meshes/Omniwheel.stl" scale="${model_scale}"/>
-            </geometry>
-        </collision>
-        <inertial>
-            <origin rpy="0 ${pi/2} 0"/>
-            <mass value="0.020"/>
-            <inertia ixx="4.05491236e-06" ixy="-2.30614871e-09" ixz="-3.59024381e-09"
-                     iyy="4.05452187e-06" iyz="2.37778687e-09"
-                     izz="5.84593279e-06" />
-        </inertial>
-    </link>
-    <link name="wheel3">
-        <visual>
-            <origin rpy="0 ${pi/2} 0"/>
-            <geometry>
-                <mesh filename="package://theclaw/urdf/meshes/Omniwheel.stl" scale="${model_scale}"/>
-            </geometry>
-        </visual>
-        <collision>
-            <origin rpy="0 ${pi/2} 0"/>
-            <geometry>
-                <mesh filename="package://theclaw/urdf/meshes/Omniwheel.stl" scale="${model_scale}"/>
-            </geometry>
-        </collision>
-        <inertial>
-            <origin rpy="0 ${pi/2} 0"/>
-            <mass value="0.020"/>
-            <inertia ixx="4.05491236e-06" ixy="-2.30614871e-09" ixz="-3.59024381e-09"
-                     iyy="4.05452187e-06" iyz="2.37778687e-09"
-                     izz="5.84593279e-06" />
-        </inertial>
-    </link>
-    <joint name="wheel1_axis" type="continuous">
+    <xacro:macro name="wheel" params="name *origin">
+        <link name="${name}_link">
+            <visual>
+                <origin rpy="0 ${pi/2} 0"/>
+                <geometry>
+                    <mesh filename="package://theclaw/urdf/meshes/Omniwheel.stl" scale="${model_scale}"/>
+                </geometry>
+            </visual>
+            <collision>
+                <origin rpy="0 ${pi/2} 0"/>
+                <geometry>
+                    <cylinder radius="0.025" length="0.025" />
+                </geometry>
+            </collision>
+            <xacro:inertial_cylinder mass="0.020" radius="0.025" length="0.025">
+                <origin rpy="0 ${pi/2} 0"/>
+            </xacro:inertial_cylinder>
+        </link>
+        <joint name="${name}_joint" type="continuous">
+            <xacro:insert_block name="origin" />
+            <parent link="base_link"/>
+            <child link="${name}_link"/>
+        </joint>
+    </xacro:macro>
+    <xacro:wheel name="wheel1">
         <origin xyz="0.077647 0 0" rpy="0 0 0"/>
-        <parent link="base_link"/>
-        <child link="wheel1"/>
-    </joint>
-    <joint name="wheel2_axis" type="continuous">
+    </xacro:wheel>
+    <xacro:wheel name="wheel2">
         <origin xyz="${cos(2*pi/3)*0.077647 - sin(2*pi/3)*0} ${sin(2*pi/3)*0.077647 + cos(2*pi/3)*0} 0" rpy="0 0 ${2*pi/3}"/>
-        <parent link="base_link"/>
-        <child link="wheel2"/>
-    </joint>
-    <joint name="wheel3_axis" type="continuous">
+    </xacro:wheel>
+    <xacro:wheel name="wheel3">
         <origin xyz="${cos(2*pi/3*2)*0.077647 - sin(2*pi/3*2)*0} ${sin(2*pi/3*2)*0.077647 + cos(2*pi/3*2)*0} 0" rpy="0 0 ${2*pi/3*2}"/>
-        <parent link="base_link"/>
-        <child link="wheel3"/>
-    </joint>
+    </xacro:wheel>
 </robot>

Commit message: jedzie

File: urdf/theclaw.urdf.xacro (robot description, xacro)
@@ -103,5 +103,5 @@
             <parent link="base_link"/>
             <child link="${name}_link"/>
-            <limit velocity="2" effort="0.01"/>
+            <limit velocity="4" effort="1"/>
         </joint>
         <transmission name="${name}_tran">

Commit message: new world

File: urdf/theclaw.urdf.xacro (robot description, xacro)
@@ -103,5 +103,5 @@
             <parent link="base_link"/>
             <child link="${name}_link"/>
-            <limit velocity="4" effort="1"/>
+            <limit velocity="2" effort="1"/>
         </joint>
         <transmission name="${name}_tran">

Commit message: jest git

File: urdf/theclaw.urdf.xacro (robot description, xacro)
@@ -103,13 +103,13 @@
             <parent link="base_link"/>
             <child link="${name}_link"/>
-            <limit velocity="2" effort="1"/>
+            <limit velocity="10.0" effort="1.0"/>
         </joint>
         <transmission name="${name}_tran">
             <type>transmission_interface/SimpleTransmission</type>
             <joint name="${name}_joint">
-                <hardwareInterface>hardware_interface/EffortJointInterface</hardwareInterface>
+                <hardwareInterface>hardware_interface/VelocityJointInterface</hardwareInterface>
             </joint>
             <actuator name="${name}_motor">
-                <hardwareInterface>hardware_interface/EffortJointInterface</hardwareInterface>
+                <hardwareInterface>hardware_interface/VelocityJointInterface</hardwareInterface>
                 <mechanicalReduction>1</mechanicalReduction>
             </actuator>

Commit message: hector

File: urdf/theclaw.urdf.xacro (robot description, xacro)
@@ -8,5 +8,5 @@
         <parent link="base_footprint"/>
         <child link="base_link"/>
-        <origin xyz="0.0 0.0 0.025" rpy=" 0 0 0"/>
+        <origin xyz="0.0 0.0 0.025" rpy="0 0 0"/>
     </joint>
     <!-- Base -->

Commit message: motors

File: urdf/theclaw.urdf.xacro (robot description, xacro)
@@ -39,4 +39,5 @@
             <parent link="base_link" />
             <child link="${name}_link" />
+            <axis xyz="0 0 1" />
         </joint>
         <transmission name="${name}_tran">

Commit message: diff drive

File: urdf/theclaw.urdf.xacro (robot description, xacro)
@@ -53,8 +53,8 @@
     </xacro:macro>
     <xacro:wheel name="wheel_left">
-        <origin xyz="0 ${-0.050-0.017/2} 0" rpy="${pi/2} 0 0" />
+        <origin xyz="0 ${-0.050-0.017/2} 0" rpy="${-pi/2} 0 0" />
     </xacro:wheel>
     <xacro:wheel name="wheel_right">
-        <origin xyz="0 ${0.050+0.017/2} 0" rpy="${-pi/2} 0 0" />
+        <origin xyz="0 ${0.050+0.017/2} 0" rpy="${pi/2} 0 ${pi}" />
     </xacro:wheel>
     <!-- Skids -->

Commit message: gripper

File: urdf/theclaw.urdf.xacro (robot description, xacro)
@@ -87,3 +87,46 @@
         <origin xyz="-0.050 0 ${-0.040+0.010+0.001}" />
     </xacro:skid>
+    <!-- Gripper -->
+    <xacro:macro name="gripper_arm" params="name *origin">
+        <link name="${name}_link">
+            <visual>
+                <origin xyz="-0.065 0.095 -0.005" rpy="0 0 ${-pi/2}"/>
+                <geometry>
+                    <mesh filename="package://theclaw/urdf/meshes/gripper_arm.stl" scale="0.001 0.001 0.001" />
+                </geometry>
+            </visual>
+            <collision>
+                <origin xyz="-0.065 0.095 -0.005" rpy="0 0 ${-pi/2}"/>
+                <geometry>
+                    <mesh filename="package://theclaw/urdf/meshes/gripper_arm.stl" scale="0.001 0.001 0.001" />
+                </geometry>
+            </collision>
+            <xacro:inertial_sphere mass="0.010" radius="0.050">
+                <origin xyz="0 0 0"/>
+            </xacro:inertial_sphere>
+        </link>
+        <joint name="${name}_joint" type="revolute">
+            <parent link="base_link" />
+            <child link="${name}_link" />
+            <xacro:insert_block name="origin" />
+            <axis xyz="0 0 1" />
+            <limit effort="0.07" velocity="1" lower="0" upper="1" />
+        </joint>
+        <transmission name="${name}_tran">
+            <type>transmission_interface/SimpleTransmission</type>
+            <joint name="${name}_joint">
+                <hardwareInterface>hardware_interface/EffortJointInterface</hardwareInterface>
+            </joint>
+            <actuator name="${name}_act">
+                <hardwareInterface>hardware_interface/EffortJointInterface</hardwareInterface>
+                <mechanicalReduction>1</mechanicalReduction>
+            </actuator>
+        </transmission>
+    </xacro:macro>
+    <xacro:gripper_arm name="gripper_arm_left">
+        <origin xyz="0.100 0.015 0.0" rpy="${pi} 0 0.75" />
+    </xacro:gripper_arm>
+    <xacro:gripper_arm name="gripper_arm_right">
+        <origin xyz="0.100 -0.015 0.0" rpy="0 0 -0.75" />
+    </xacro:gripper_arm>
 </robot>

Commit message: grabber pid

File: urdf/theclaw.urdf.xacro (robot description, xacro)
@@ -111,5 +111,5 @@
             <xacro:insert_block name="origin" />
             <axis xyz="0 0 1" />
-            <limit effort="0.07" velocity="1" lower="0" upper="1" />
+            <limit effort="0.07" velocity="10" lower="0" upper="1" />
         </joint>
         <transmission name="${name}_tran">
